Commit message: second

File: arm_description/urdf/arm.urdf.xacro (robot description, xacro)
@@ -347,3 +347,62 @@
     </inertial>
   </link>
+   <gazebo>
+    <plugin filename="ign_ros2_control-system" name="ign_ros2_control::IgnitionROS2ControlPlugin">
+    <parameters>$(find arm_control)/config/arm_controllers.yaml</parameters>
+      <controller_manager_prefix_node_name>controller_manager</controller_manager_prefix_node_name>
+    </plugin>
+  </gazebo>
+  <ros2_control name="HardwareInterface_Ignition" type="system">
+    <hardware>
+      <plugin>ign_ros2_control/IgnitionSystem</plugin>
+    </hardware>
+     <joint name="j0">
+        <command_interface name="position"/>
+        <state_interface name="position">
+            <param name="initial_value">0.0</param>
+        </state_interface>
+        <state_interface name="velocity">
+            <param name="initial_value">0.0</param>
+        </state_interface>
+        <state_interface name="effort">
+            <param name="initial_value">0.0</param>
+        </state_interface>
+    </joint>
+    <joint name="j1">
+        <command_interface name="position"/>
+        <state_interface name="position">
+            <param name="initial_value">0.0</param>
+        </state_interface>
+        <state_interface name="velocity">
+            <param name="initial_value">0.0</param>
+        </state_interface>
+        <state_interface name="effort">
+            <param name="initial_value">0.0</param>
+        </state_interface>
+    </joint>
+    <joint name="j2">
+        <command_interface name="position"/>
+        <state_interface name="position">
+            <param name="initial_value">0.0</param>
+        </state_interface>
+        <state_interface name="velocity">
+            <param name="initial_value">0.0</param>
+        </state_interface>
+        <state_interface name="effort">
+            <param name="initial_value">0.0</param>
+        </state_interface>
+    </joint>
+    <joint name="j3">
+        <command_interface name="position"/>
+        <state_interface name="position">
+            <param name="initial_value">0.0</param>
+        </state_interface>
+        <state_interface name="velocity">
+            <param name="initial_value">0.0</param>
+        </state_interface>
+        <state_interface name="effort">
+            <param name="initial_value">0.0</param>
+        </state_interface>
+    </joint>
+  </ros2_control>
 </robot>

Commit message: punto 4a

File: arm_description/urdf/arm.urdf.xacro (robot description, xacro)
@@ -347,4 +347,19 @@
     </inertial>
   </link>
+  <!-- <joint name="camera_joint" type="fixed">
+      <parent link="base_link"/>
+      <child link="camera_link"/>
+      <origin xyz="0.0 0 0.00" rpy="0.0 -1.57 0"/>
+  </joint>
+  <link name="camera_link">
+      <visual>
+          <geometry>
+              <box size="0.010 0.01000003 0.01000003"/>
+          </geometry>
+          <material name="red"/>
+      </visual>
+  </link> -->
+  <xacro:include filename="$(find arm_description)/urdf/cam_tot.xacro"/>
+  <xacro:my_camera parent_link="base_link"/>
   <gazebo>
     <plugin filename="ign_ros2_control-system" name="ign_ros2_control::IgnitionROS2ControlPlugin">
@@ -353,9 +368,14 @@
     </plugin>
   </gazebo>
+  <xacro:include filename="$(find arm_description)/urdf/arm_hardware_interface.xacro"/>
   <ros2_control name="HardwareInterface_Ignition" type="system">
     <hardware>
       <plugin>ign_ros2_control/IgnitionSystem</plugin>
     </hardware>
-     <joint name="j0">
+    <xacro:joint_ros2_control name="j0"/>
+    <xacro:joint_ros2_control name="j1"/>
+    <xacro:joint_ros2_control name="j2"/>
+    <xacro:joint_ros2_control name="j3"/>
+     <!-- <joint name="j0">
         <command_interface name="position"/>
         <state_interface name="position">
@@ -404,5 +424,5 @@
             <param name="initial_value">0.0</param>
         </state_interface>
-    </joint>
+    </joint> -->
   </ros2_control>
 </robot>
